File: OpenHardwareExG_ActiveElectrodeAdapter.sch (KiCad schematic (older format))
At the start: 18 parts, among them P1 CONN_01X03, P10 CONN_01X03, P11 CONN_01X03, P12 CONN_01X03, P13 CONN_01X03, P14 CONN_01X03, P15 CONN_01X03, P16 CONN_01X03, P17 CONN_01X20, P18 CONN_01X18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

Commit message: most PCB routing done.
Parts:
- P1, P10, P11, P12, P13, P14, P15, P16, P2, P3, P4, P5, P6, P7, P8, P9: footprint (none) -> active_electrode_connectors:DF50A-3P-1V
- P17: footprint (none) -> Pin_Headers:Pin_Header_Straight_1x20
- P18: footprint (none) -> Pin_Headers:Pin_Header_Straight_1x18
Changed lines of the file:
@@
 F 0 "P18" H 8350 5000 50  0000 C CNN
 F 1 "CONN_01X18" V 8450 4050 50  0000 C CNN
-F 2 "" H 8350 4050 50  0000 C CNN
+F 2 "Pin_Headers:Pin_Header_Straight_1x18" H 8350 4050 50  0001 C CNN
 F 3 "" H 8350 4050 50  0000 C CNN
 	1    8350 4050
@@
 F 0 "P4" H 2500 5100 50  0000 C CNN
 F 1 "CONN_01X03" V 2600 4900 50  0000 C CNN
-F 2 "" H 2500 4900 50  0000 C CNN
+F 2 "active_electrode_connectors:DF50A-3P-1V" H 2500 4900 50  0001 C CNN
 F 3 "" H 2500 4900 50  0000 C CNN
 	1    2500 4900
@@
 F 0 "P3" H 2500 4500 50  0000 C CNN
 F 1 "CONN_01X03" V 2600 4300 50  0000 C CNN
-F 2 "" H 2500 4300 50  0000 C CNN
+F 2 "active_electrode_connectors:DF50A-3P-1V" H 2500 4300 50  0001 C CNN
 F 3 "" H 2500 4300 50  0000 C CNN
 	1    2500 4300
@@
 F 0 "P2" H 2500 3900 50  0000 C CNN
 F 1 "CONN_01X03" V 2600 3700 50  0000 C CNN
-F 2 "" H 2500 3700 50  0000 C CNN
+F 2 "active_electrode_connectors:DF50A-3P-1V" H 2500 3700 50  0001 C CNN
 F 3 "" H 2500 3700 50  0000 C CNN
 	1    2500 3700
@@
 F 0 "P1" H 2500 3300 50  0000 C CNN
 F 1 "CONN_01X03" V 2600 3100 50  0000 C CNN
-F 2 "" H 2500 3100 50  0000 C CNN
+F 2 "active_electrode_connectors:DF50A-3P-1V" H 2500 3100 50  0001 C CNN
 F 3 "" H 2500 3100 50  0000 C CNN
 	1    2500 3100
@@
 F 0 "P8" H 3500 5100 50  0000 C CNN
 F 1 "CONN_01X03" V 3600 4900 50  0000 C CNN
-F 2 "" H 3500 4900 50  0000 C CNN
+F 2 "active_electrode_connectors:DF50A-3P-1V" H 3500 4900 50  0001 C CNN
 F 3 "" H 3500 4900 50  0000 C CNN
 	1    3500 4900
@@
 F 0 "P7" H 3500 4500 50  0000 C CNN
 F 1 "CONN_01X03" V 3600 4300 50  0000 C CNN
-F 2 "" H 3500 4300 50  0000 C CNN
+F 2 "active_electrode_connectors:DF50A-3P-1V" H 3500 4300 50  0001 C CNN
 F 3 "" H 3500 4300 50  0000 C CNN
 	1    3500 4300
@@
 F 0 "P6" H 3500 3900 50  0000 C CNN
 F 1 "CONN_01X03" V 3600 3700 50  0000 C CNN
-F 2 "" H 3500 3700 50  0000 C CNN
+F 2 "active_electrode_connectors:DF50A-3P-1V" H 3500 3700 50  0001 C CNN
 F 3 "" H 3500 3700 50  0000 C CNN
 	1    3500 3700
@@
 F 0 "P5" H 3500 3300 50  0000 C CNN
 F 1 "CONN_01X03" V 3600 3100 50  0000 C CNN
-F 2 "" H 3500 3100 50  0000 C CNN
+F 2 "active_electrode_connectors:DF50A-3P-1V" H 3500 3100 50  0001 C CNN
 F 3 "" H 3500 3100 50  0000 C CNN
 	1    3500 3100
@@
 F 0 "P12" H 4500 5100 50  0000 C CNN
 F 1 "CONN_01X03" V 4600 4900 50  0000 C CNN
-F 2 "" H 4500 4900 50  0000 C CNN
+F 2 "active_electrode_connectors:DF50A-3P-1V" H 4500 4900 50  0001 C CNN
 F 3 "" H 4500 4900 50  0000 C CNN
 	1    4500 4900
@@
 F 0 "P11" H 4500 4500 50  0000 C CNN
 F 1 "CONN_01X03" V 4600 4300 50  0000 C CNN
-F 2 "" H 4500 4300 50  0000 C CNN
+F 2 "active_electrode_connectors:DF50A-3P-1V" H 4500 4300 50  0001 C CNN
 F 3 "" H 4500 4300 50  0000 C CNN
 	1    4500 4300
@@
 F 0 "P10" H 4500 3900 50  0000 C CNN
 F 1 "CONN_01X03" V 4600 3700 50  0000 C CNN
-F 2 "" H 4500 3700 50  0000 C CNN
+F 2 "active_electrode_connectors:DF50A-3P-1V" H 4500 3700 50  0001 C CNN
 F 3 "" H 4500 3700 50  0000 C CNN
 	1    4500 3700
@@
 F 0 "P9" H 4500 3300 50  0000 C CNN
 F 1 "CONN_01X03" V 4600 3100 50  0000 C CNN
-F 2 "" H 4500 3100 50  0000 C CNN
+F 2 "active_electrode_connectors:DF50A-3P-1V" H 4500 3100 50  0001 C CNN
 F 3 "" H 4500 3100 50  0000 C CNN
 	1    4500 3100
@@
 F 0 "P16" H 5500 5100 50  0000 C CNN
 F 1 "CONN_01X03" V 5600 4900 50  0000 C CNN
-F 2 "" H 5500 4900 50  0000 C CNN
+F 2 "active_electrode_connectors:DF50A-3P-1V" H 5500 4900 50  0001 C CNN
 F 3 "" H 5500 4900 50  0000 C CNN
 	1    5500 4900
@@
 F 0 "P15" H 5500 4500 50  0000 C CNN
 F 1 "CONN_01X03" V 5600 4300 50  0000 C CNN
-F 2 "" H 5500 4300 50  0000 C CNN
+F 2 "active_electrode_connectors:DF50A-3P-1V" H 5500 4300 50  0001 C CNN
 F 3 "" H 5500 4300 50  0000 C CNN
 	1    5500 4300
@@
 F 0 "P14" H 5500 3900 50  0000 C CNN
 F 1 "CONN_01X03" V 5600 3700 50  0000 C CNN
-F 2 "" H 5500 3700 50  0000 C CNN
+F 2 "active_electrode_connectors:DF50A-3P-1V" H 5500 3700 50  0001 C CNN
 F 3 "" H 5500 3700 50  0000 C CNN
 	1    5500 3700
@@
 F 0 "P13" H 5500 3300 50  0000 C CNN
 F 1 "CONN_01X03" V 5600 3100 50  0000 C CNN
-F 2 "" H 5500 3100 50  0000 C CNN
+F 2 "active_electrode_connectors:DF50A-3P-1V" H 5500 3100 50  0001 C CNN
 F 3 "" H 5500 3100 50  0000 C CNN
 	1    5500 3100
@@
 F 0 "P17" H 7000 5000 50  0000 C CNN
 F 1 "CONN_01X20" V 7100 3950 50  0000 C CNN
-F 2 "" H 7000 3950 50  0000 C CNN
+F 2 "Pin_Headers:Pin_Header_Straight_1x20" H 7000 3950 50  0001 C CNN
 F 3 "" H 7000 3950 50  0000 C CNN
 	1    7000 3950

Commit message: add RLD
Parts:
- added P19: CONN_01X01, Pin_Headers:Pin_Header_Straight_1x01, symbol CONN_01X01
Connections:
- net RLD: now also P19.1 (P1)
Changed lines of the file:
@@
 	1    0    0    1
 $EndComp
+$Comp
+L CONN_01X01 P19
+U 1 1 56C874FE
+P 1500 4000
+F 0 "P19" H 1500 4100 50  0000 C CNN
+F 1 "CONN_01X01" V 1600 4000 50  0000 C CNN
+F 2 "Pin_Headers:Pin_Header_Straight_1x01" H 1500 4000 50  0001 C CNN
+F 3 "" H 1500 4000 50  0000 C CNN
+	1    1500 4000
+	1    0    0    -1
+$EndComp
+Wire Wire Line
+	1000 4000 1300 4000
+Text Label 1000 4000 0    60   ~ 0
+RLD
 $EndSCHEMATC
